File: PCB/KlipperToolboard/KlipperToolboard.kicad_pcb (KiCad board)
At the start: 4 copper layers, 45 x 48 mm, 79 parts, among them J1 Endstop, J10 Conn_01x04_Male, J2 Conn_01x04, J3 HeaterThermistor, J4 PartFan, J5 HeaterFan, J6 Heater, J7 Conn_01x03, J8 Conn_01x02, J9 Stepper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

Commit message: Tweaks and 3d models
Parts:
- J4, J5, J6: footprint TerminalBlock_TE-Connectivity:TerminalBlock_TE_282834-2_1x02_P2.54mm_Horizontal -> KlipperToolboard:TerminalBlock_TE_282834-2_1x02_P2.54mm_Horizontal
