File: PCB/HuvudTiny/Huvud.sch (KiCad schematic (older format))
At the start: 98 parts, among them J10 JST_PH, J12 USB_Micro-B_Molex-105017-0001, J2 DBG, J3 THERM, J4 FAN0, J5 FAN1, J6 Heater, J7 Endstop, J8 Conn_01x02, J9 STEPPER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

Commit message: v0.44, v0.45
Parts:
- removed C26: 0.1uF, Capacitor_SMD:C_0402_1005Metric, symbol Device:C_Small
- removed D7: B5819W, Diode_SMD:D_SOD-123, symbol Device:D_Schottky
- removed J8: Conn_01x02, Connector_Molex:Molex_Micro-Fit_3.0_43650-0200_1x02_P3.00mm_Horizontal, symbol Connector_Generic:Conn_01x02
- removed L2: 22uH, Inductor_SMD:L_0805_2012Metric, symbol pspice:INDUCTOR
- removed L3: 10uH, Inductor_SMD:L_Sunlord_MWSA0518_5.4x5.2mm, symbol Device:L_Core_Iron
- removed R32: 160k, Resistor_SMD:R_0402_1005Metric, symbol Device:R_Small
- removed R33: 33k, Resistor_SMD:R_0402_1005Metric, symbol Device:R_Small
- removed U1: TPS54331DR, Package_SO:SOIC-8_3.9x4.9mm_P1.27mm, symbol Regulator_Switching:TPS54233
- added 3.3, GND1, GND2, PB10, PB11, TP1, TP2, TP3, TP4, TP5, TP6, VIN1: TestPoint, TestPoint:TestPoint_Pad_D1.0mm, symbol Connector:TestPoint
- added C32: 10uF, Capacitor_SMD:C_0805_2012Metric, symbol Device:C_Small
- added J1: Conn_02x02_Odd_Even, Connector_Molex:Molex_Micro-Fit_3.0_43045-0400_2x02_P3.00mm_Horizontal, symbol Connector_Generic:Conn_02x02_Top_Bottom
- added L4: 10uH/max 145mOhm 2A, Inductor_SMD:L_Sunlord_MWSA0518_5.4x5.2mm, symbol Device:L_Core_Iron
- added NT1: Net-Tie_2, NetTie:NetTie-2_SMD_Pad0.5mm, symbol Device:Net-Tie_2
- added R37: 10k, Resistor_SMD:R_0402_1005Metric, symbol Device:R_Small
- added R38, R40: 100k, Resistor_SMD:R_0402_1005Metric, symbol Device:R_Small
- added R39, R41: 22k, Resistor_SMD:R_0402_1005Metric, symbol Device:R_Small
- added U3: TPS54308, Package_TO_SOT_SMD:SOT-23-6, symbol Regulator_Switching:TPS54308
- C1, C27: LCSC (none) -> C23733
- C10: LCSC (none) -> C1525
- C14: value 2.2nF -> 10uF; footprint Capacitor_SMD:C_0402_1005Metric -> Capacitor_SMD:C_0805_2012Metric; LCSC C1531 -> C15850
- C15: value 22pF/35V -> 10uF; footprint Capacitor_SMD:C_0402_1005Metric -> Capacitor_SMD:C_0805_2012Metric; LCSC C1555 -> C15850
- C16: value 22nf/50V -> 0.1uF/35V; LCSC C21122 -> C14663
- C20: value 10uF/35V -> 0.1uF/35V; footprint Capacitor_SMD:C_1206_3216Metric -> Capacitor_SMD:C_0603_1608Metric; LCSC C13585 -> C14663
- C21: value 0.1uF -> 68pF; LCSC (none) -> C14441
- C22: value 10uF -> 10uF/35V; footprint Capacitor_SMD:C_0603_1608Metric -> Capacitor_SMD:C_1210_3225Metric; LCSC C19702 -> C13585
- C23: value 10uF -> 4.7uF; footprint Capacitor_SMD:C_0603_1608Metric -> Capacitor_SMD:C_0402_1005Metric; LCSC (none) -> C23733
- C3, C6, C7: value 0.1uF -> 0.1uF/35V
- C4: LCSC C19666 -> C23733
- C9: LCSC C14663 -> C1525
- D5: value LEDRED -> LEDGR; footprint LED_SMD:LED_0603_1608Metric -> LED_SMD:LED_0402_1005Metric; LCSC C2286 -> C74338
- H1, H2, H3, H4: footprint MountingHole:MountingHole_3.2mm_M3_Pad -> MountingHole:MountingHole_3.2mm_M3_Pad_Via
- Q3: value AO3400A -> AON7524; footprint Package_TO_SOT_SMD:SOT-23 -> Huvud:DFN-8-1EP_3x3mm_P0.65mm_EP1.7x2.05mm; symbol Transistor_FET:2N7002 -> Huvud:AON7418; LCSC C20917 -> C431195
- R10, R12, R13, R14, R15, R21: LCSC (none) -> C25744
- R17, R18, R24: value 20k -> 22k; LCSC C25765 -> C25768
- R2: value 4.7k -> 2.2k; LCSC C25900 -> C25879
- R27: value 1.5k -> 2.2k; LCSC C25867 -> C25879
- R29: value 4.7k -> 2.2k; LCSC (none) -> C25879
- R30: value 10k -> 22; LCSC (none) -> C25092
- R31: value 3.3k -> 22; LCSC C25890 -> C25092
- R4, R7: value 0.110 -> 0.110 1%; LCSC C247458 -> C327071
Connections:
- net +3V3: now also C14.1, C15.1, R30.1, 3.3.1, C32.1, L4.2, TP6.1; no longer C11.2, C22.2, C23.2, R30.2
- net AREF: now also C11.2, C23.2
- net BOOT0: now also TP1.1; no longer J2.1 (Pin_1)
- net CANH: now also J1.2 (Pin_2)
- net CANL: now also J1.1 (Pin_1)
- net GND: now also C15.2, C16.2, Q3.1 (S), C32.2, GND1.1, GND2.1, J1.3 (Pin_3), NT1.1, R37.1, R39.1, R41.1, U3.1 (GND); no longer C11.1, C15.1, C16.1, C20.1, C23.1, Q3.2 (S), R31.1
- net GNDA: now also C11.1, C23.1, NT1.2
- net ST_A1: now also J9.2 (Pin_2), TP3.1; no longer J9.3 (Pin_3)
- net ST_A2: now also J9.1 (Pin_1), TP2.1; no longer J9.4 (Pin_4)
- net ST_B1: now also J9.3 (Pin_3), TP4.1; no longer J9.2 (Pin_2)
- net ST_B2: now also J9.4 (Pin_4), TP5.1; no longer J9.1 (Pin_1)
- net VDC: now also C16.1, C22.2, J1.4 (Pin_4), R38.2, U3.3 (VIN), VIN1.1; no longer C20.2
- net BOOT1: now reaches U5.20 (PB2)
- net BOOT1: now also J2.1 (Pin_1), R37.2
- net at U5.21 (PB10): now also PB10.1
- net at U5.22 (PB11): now also PB11.1
- net at R28.2: now also Q3.2 (G); no longer Q3.1 (G)
- net at C21.2: now also R29.1
- net at R31.2: now also R30.2; no longer R30.1
- net at R29.2: now also R31.1, R40.2; no longer C15.2
- net at C21.1: now also R40.1, R41.2, U3.4 (FB)
- new net: C20.1, L4.1, U3.2 (SW)
- new net: R38.1, R39.2, U3.5 (EN)
- new net: C20.2, U3.6 (BOOT)
- no-connect marks 22 -> 19
Other:
- note added: "0.45"
- note added: "Alt: RU3040M2"
- note added: "Alt: \nTPS54202\nTPS54302"
- note added: "Or 2x 22uF"
- note removed: "TODO:\nMP2359 is an alternative smaller SW controller"
- moved on the sheet: C2, D4, H1, H2, H3, H4, J7, J9, R19, R23, R36

Commit message: Minor tweaks to the layout. Added some text on the back size
Parts:
- J1: LCSC (none) -> C122413
Changed lines of the file:
@@
 F 2 "Connector_Molex:Molex_Micro-Fit_3.0_43045-0400_2x02_P3.00mm_Horizontal" H 7150 4050 50  0001 C CNN
 F 3 "~" H 7150 4050 50  0001 C CNN
+F 4 "C122413" H 7150 4050 50  0001 C CNN "LCSC"
 	1    7150 4050
 	-1   0    0    -1
