File: PCB/HuvudTiny/Huvud.kicad_pcb (KiCad board)
At the start: 4 copper layers, 42 x 42 mm, 113 parts, among them J1 Conn_02x02_Odd_Even, J12 USB_Micro-B_Molex-105017-0001, J2 DBG, J3 THERM, J4 FAN0, J5 FAN1, J6 Heater, J7 Endstop, J9 STEPPER, Q1 AO3400A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

Commit message: Tweaks
Parts:
- added C26: 22pF, Capacitor_SMD:C_0402_1005Metric, F.Cu at (203.7, 106.9)
- added C29: 22pF, Capacitor_SMD:C_0402_1005Metric, F.Cu at (203.7, 105.0)
- R1: value 4.7k -> 10k
- moved R11 3.66 mm to (200.7, 103.4)
- moved D6 0.28 mm to (202.7, 103.2)
Routing:
- net GND: track 146.8 -> 151.8 mm, vias 100 -> 98
- net Net-(D6-Pad1): track 2.27 -> 1.45 mm
- net CANH: track 24.7 -> 24.1 mm
