File: PCB/CanDist/CanCape.kicad_pcb (KiCad board)
At the start: 2 copper layers, 36 x 66 mm, 15 parts, among them J1 Conn_01x02, J10 Conn_01x02, J11 Conn_01x02, J2 Conn_02x02_Top_Bottom, J3 Conn_02x02_Top_Bottom, J4 Conn_02x02_Top_Bottom, J5 Conn_02x02_Top_Bottom, J6 Conn_02x02_Top_Bottom, J7 Conn_02x02_Top_Bottom, J8 Conn_02x02_Top_Bottom, J9 Conn_02x02_Top_Bottom

Commit message: Added step file for Huvud v0.62
Parts:
- removed F1: Fuse, cancape:3544-2_FuseHolder
- added H1: MountingHole, MountingHole:MountingHole_3.2mm_M3_Pad_Via, F.Cu at (110.4, 52.4)
- added H2: MountingHole, MountingHole:MountingHole_3.2mm_M3_Pad_Via, F.Cu at (187.4, 52.4)
- added J12: Conn_01x01, Connector_PinHeader_2.54mm:PinHeader_1x01_P2.54mm_Vertical, F.Cu at (155.8, 60.2)
- added J13: Conn_01x01, Connector_PinHeader_2.54mm:PinHeader_1x01_P2.54mm_Vertical, F.Cu at (166.8, 60.2)
- added J14: Conn_02x02_Top_Bottom, Connector_Molex:Molex_Micro-Fit_3.0_43045-0400_2x02_P3.00mm_Horizontal, F.Cu at (147.0, 51.4)
- added J15: Conn_02x02_Top_Bottom, Connector_Molex:Molex_Micro-Fit_3.0_43045-0400_2x02_P3.00mm_Horizontal, F.Cu at (158.0, 51.4)
- added J16: Conn_02x02_Top_Bottom, Connector_Molex:Molex_Micro-Fit_3.0_43045-0400_2x02_P3.00mm_Horizontal, F.Cu at (169.0, 51.4)
- F2: footprint cancape:3544-2_FuseHolder -> cancape:KEYSTONE-3568
- J11: value Conn_01x02 -> Conn_02x02_Top_Bottom; footprint Connector_PinHeader_2.54mm:PinHeader_1x02_P2.54mm_Vertical -> Connector_Molex:Molex_Micro-Fit_3.0_43045-0400_2x02_P3.00mm_Horizontal
- J6, J7: value Conn_02x02_Top_Bottom -> Conn_01x02; footprint Connector_Molex:Molex_Micro-Fit_3.0_43045-0412_2x02_P3.00mm_Vertical -> Connector_JST:JST_XH_B2B-XH-A_1x02_P2.50mm_Vertical
- J8, J9: value Conn_02x02_Top_Bottom -> Conn_01x01; footprint Connector_Molex:Molex_Micro-Fit_3.0_43045-0412_2x02_P3.00mm_Vertical -> Connector_PinHeader_2.54mm:PinHeader_1x01_P2.54mm_Vertical
- R2: footprint Resistor_SMD:R_0603_1608Metric -> Resistor_THT:R_Axial_DIN0207_L6.3mm_D2.5mm_P7.62mm_Horizontal
- moved J1 75.7 mm to (120.4, 54.3), turned to 270 degrees
- moved F2 74.6 mm to (129.9, 48.9), turned to 270 degrees
- moved J10 73.8 mm to (181.0, 55.8), turned to 180 degrees
- moved R1 72.9 mm to (177.5, 56.1)
- moved J7 66.0 mm to (179.6, 48.4)
- moved J11 65.3 mm to (136.0, 51.4), turned to 0 degrees
- moved R2 65.2 mm to (177.5, 52.5)
- moved J6 61.8 mm to (120.4, 48.4)
- moved J2 59.7 mm to (136.0, 51.4), turned to 0 degrees
- moved J3 46.5 mm to (147.0, 51.4), turned to 0 degrees
- moved J4 35.2 mm to (158.0, 51.4), turned to 0 degrees
- moved J5 28.3 mm to (169.0, 51.4), turned to 0 degrees
- moved J8 26.2 mm to (133.8, 60.2), turned to 0 degrees
- moved J9 17.9 mm to (144.8, 60.2), turned to 0 degrees
Connections:
- F2 pad 1: Net-(F1-Pad1) -> /VIN
- F2 pad 2: Net-(F2-Pad2) -> /VINF
- J1 pad 1: GND -> /VIN
- J1 pad 2: Net-(F1-Pad1) -> GND
- J10 pad 2: CAN2H -> CANH
- J11 pad 1: Net-(J11-Pad1) -> CANL
- J11 pad 2: CAN2H -> CANH
- J2 pad 1: CAN2L -> CANL
- J2 pad 2: CAN2H -> CANH
- J2 pad 4: Net-(F2-Pad2) -> /VINF
- J3 pad 1: CAN2L -> CANL
- J3 pad 2: CAN2H -> CANH
- J3 pad 4: Net-(F2-Pad2) -> /VINF
- J4 pad 1: CAN2L -> CANL
- J4 pad 2: CAN2H -> CANH
- J4 pad 4: Net-(F2-Pad2) -> /VINF
- J5 pad 1: CAN2L -> CANL
- J5 pad 2: CAN2H -> CANH
- J5 pad 4: Net-(F2-Pad2) -> /VINF
- J6 pad 1: CAN2L -> CANL
- J6 pad 2: CAN2H -> CANH
- J7 pad 1: CAN2L -> CANL
- J7 pad 2: CAN2H -> CANH
- J8 pad 1: CAN2L -> GND
- J9 pad 1: CAN2L -> GND
- R1 pad 1: CAN2L -> CANL
- R2 pad 1: CAN2L -> CANL
- R2 pad 2: Net-(J11-Pad1) -> Net-(J10-Pad1)
Routing:
- net CAN2L: track 116.9 -> 0.00 mm
- net CAN2H: track 112.5 -> 0.00 mm
- net CANL: track 0.00 -> 76.4 mm
- net CANH: track 0.00 -> 75.2 mm
- net Net-(J11-Pad1): track 6.83 -> 0.00 mm
- net Net-(J10-Pad1): track 2.84 -> 7.18 mm
- added copper zone on F.Cu, net /VIN
- added copper zone on F.Cu, net /VINF
- removed copper zone on F.Cu, net Net-(F1-Pad1)
- removed copper zone on F.Cu, net Net-(F1-Pad2)
- removed copper zone on F.Cu, net Net-(F2-Pad2)
Other:
- board size 36 x 66 mm -> 88.9 x 20 mm
- board text added: "H"
- board text added: "L"
- board text added: "TERM"
- board text added: "v1.0"
- board text removed: "A"
- board text removed: "B"
- board text removed: "v0.2"
