File: PCB/CanHatFd/CanHat.kicad_pcb (KiCad board)
At the start: 2 copper layers, 65 x 44 mm, 39 parts, among them J1 Raspberry_Pi_2_3, J10 Conn_02x02_Top_Bottom, J11 Conn_02x02_Top_Bottom, J12 Conn_02x02_Top_Bottom, J13 Conn_02x02_Top_Bottom, J14 Conn_01x02, J15 Conn_01x04, J2 Conn_01x02, J3 Conn_02x02_Top_Bottom, J4 Conn_02x02_Top_Bottom, J5 Conn_02x02_Top_Bottom, J6 Conn_02x02_Top_Bottom, J7 Conn_01x02, J8 Conn_01x02, U1 MCP2517FD-xSL, U2 AP1117-33, U3 MCP2558FD-xSN, Y1 Crystal_GND24

Commit message: Added step file for Huvud v0.62
Parts:
- removed J10, J11, J12, J13: Conn_02x02_Top_Bottom, Connector_Molex:Molex_Micro-Fit_3.0_43045-0412_2x02_P3.00mm_Vertical
- removed J14: Conn_01x02, Connector_PinHeader_2.54mm:PinHeader_1x02_P2.54mm_Vertical
- removed R3: 120R, Resistor_SMD:R_0603_1608Metric
- removed U3: MCP2558FD-xSN, Package_SO:SOIC-8_3.9x4.9mm_P1.27mm
- added U4: MCP2562-E-SN, Package_SO:SOIC-8_3.9x4.9mm_P1.27mm, F.Cu at (153.8, 112.2)
- moved C3 8.67 mm to (150.8, 117.4), turned to 0 degrees
Connections:
- C3 pad 1: +3V3 -> 5VPI
- C8 pad 2: 5VPI -> +3V3
Routing:
- net CANL: track 121.8 -> 56.9 mm, vias 2 -> 0
- net CANH: track 128.2 -> 66.1 mm
- net GND: track 52.2 -> 57.0 mm, vias 41 -> 32
- net Net-(J14-Pad1): track 3.44 -> 0.00 mm
- net +3V3: track 47.6 -> 44.9 mm
- net 5VPI: track 80.1 -> 79.1 mm, vias 0 -> 2
- net Net-(J8-Pad1): track 4.49 -> 5.45 mm
- net /TX: vias 2 -> 0
Other:
- board size 65 x 44 mm -> 65 x 30 mm
- rule pad_to_mask_clearance: 0.051 -> 0.025
