File: PCB/HuvudCanUSB/CanTactDist.kicad_pcb (KiCad board)
At the start: 2 copper layers, 37 x 15 mm, 41 parts, among them J1 Conn_01x03, J12 USB_Micro-B_Molex-105017-0001, J4 Conn_01x02, U1 STM32F042C6Tx, U2 XC6206P332MR, U3 USBLC6-2SC6, U6 SN65HVD230

Commit message: Added step file for Huvud v0.62
Other:
- rule pad_to_mask_clearance: 0.051 -> 0.027
Changed lines of the file:
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@@
     (pad_size 1.524 1.524)
     (pad_drill 0.762)
-    (pad_to_mask_clearance 0.051)
+    (pad_to_mask_clearance 0.027)
     (solder_mask_min_width 0.25)
     (aux_axis_origin 0 0)
